File: DISPLAY.kicad_sch (KiCad schematic)
At the start: 0 parts

Commit message: Display
Parts:
- added U4: ~, symbol HYBRID_SYMBOLS:MXS_STRADA
Connections:
- new net 12V: U4.1 (VIN)
- new net CAN-B-H: U4.8 (CAN-H)
- new net CAN-B-L: U4.9 (CAN-L)
- new net GND: U4.2 (GND)
Changed lines of the file:
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@@
 	(generator_version "9.0")
 	(paper "A4")
+	(wire
+		(pts
+			(xy 82.55 50.8) (xy 82.55 55.88)
+		)
+		(stroke
+			(width 0)
+			(type default)
+		)
+	)
+	(wire
+		(pts
+			(xy 83.82 73.66) (xy 87.63 73.66)
+		)
+		(stroke
+			(width 0)
+			(type default)
+		)
+	)
+	(wire
+		(pts
+			(xy 82.55 55.88) (xy 87.63 55.88)
+		)
+		(stroke
+			(width 0)
+			(type default)
+		)
+	)
+	(wire
+		(pts
+			(xy 119.38 60.96) (xy 114.3 60.96)
+		)
+		(stroke
+			(width 0)
+			(type default)
+		)
+	)
+	(wire
+		(pts
+			(xy 101.6 81.28) (xy 101.6 78.74)
+		)
+		(stroke
+			(width 0)
+			(type default)
+		)
+	)
+	(hierarchical_label "CAN-B-L"
+		(shape bidirectional)
+		(at 119.38 60.96 0)
+		(effects
+			(font
+				(size 1.27 1.27)
+			)
+			(justify left)
+		)
+	)
+	(hierarchical_label "GND"
+		(shape passive)
+		(at 101.6 81.28 270)
+		(effects
+			(font
+				(size 1.27 1.27)
+			)
+			(justify right)
+		)
+	)
+	(hierarchical_label "12V"
+		(shape input)
+		(at 82.55 50.8 90)
+		(effects
+			(font
+				(size 1.27 1.27)
+			)
+			(justify left)
+		)
+	)
+	(hierarchical_label "CAN-B-H"
+		(shape bidirectional)
+		(at 83.82 73.66 180)
+		(effects
+			(font
+				(size 1.27 1.27)
+			)
+			(justify right)
+		)
+	)
+	(symbol
+		(lib_name "MXS_STRADA_1")
+		(lib_id "HYBRID_SYMBOLS:MXS_STRADA")
+		(at 101.6 64.77 0)
+		(unit 1)
+		(exclude_from_sim no)
+		(in_bom yes)
+		(on_board yes)
+		(dnp no)
+		(fields_autoplaced yes)
+		(property "Reference" "U4"
+			(at 100.965 45.72 0)
+			(effects
+				(font
+					(size 1.27 1.27)
+				)
+			)
+		)
+		(property "Value" "~"
+			(at 100.965 48.26 0)
+			(effects
+				(font
+					(size 1.27 1.27)
+				)
+			)
+		)
+		(property "Footprint" ""
+			(at 101.6 64.77 0)
+			(effects
+				(font
+					(size 1.27 1.27)
+				)
+				(hide yes)
+			)
+		)
+		(property "Datasheet" ""
+			(at 101.6 64.77 0)
+			(effects
+				(font
+					(size 1.27 1.27)
+				)
+				(hide yes)
+			)
+		)
+		(property "Description" ""
+			(at 101.6 64.77 0)
+			(effects
+				(font
+					(size 1.27 1.27)
+				)
+				(hide yes)
+			)
+		)
+		(pin "3"
+		)
+		(pin "2"
+		)
+		(pin "7"
+		)
+		(pin "6"
+		)
+		(pin "12"
+		)
+		(pin "1"
+		)
+		(pin "9"
+		)
+		(pin "10"
+		)
+		(pin "5"
+		)
+		(pin "4"
+		)
+		(pin "11"
+		)
+		(pin "8"
+		)
+		(pin "13"
+		)
+		(pin "14"
+		)
+		(instances
+			(project ""
+				(path "/6f31461c-1ce3-4669-a628-d5dc5fed8080/182b60d9-b4a1-43fd-9b61-402a125a94b2"
+					(reference "U4")
+					(unit 1)
+				)
+			)
+		)
+	)
 )
