File: SKIDOO ELECTRICAL.kicad_sch (KiCad schematic)
At the start: 0 parts

Commit message: Power Supply
Parts:
- added BT1: 12V BATTERY, symbol Device:Battery_Cell
- added F1: MAIN FUSE, symbol Device:Fuse
- added F2, F3, F4, F5: FUSE, symbol Device:Fuse
- added K1: SKIDOO ON-BOARD ELECTRICAL RELAY, Relay_THT:Relay_SPDT_Fujitsu_FTR-LYCA005x_FormC_Vertical, symbol Relay:Fujitsu_FTR-LYCA005x
- added K2: ACCESSORIES RELAY, Relay_THT:Relay_SPDT_Fujitsu_FTR-LYCA005x_FormC_Vertical, symbol Relay:Fujitsu_FTR-LYCA005x
- added SW1: SW_DPST, symbol Switch:SW_DPST
- added U1, U2: ~, symbol HYBRID_SYMBOLS:BRB
Connections:
- new net: U1., U2.
- new net: SW1.3, U1.
- new net: BT1.1 (+), SW1.1
- new net: F1.2, F3.1, F4.1, F5.2
- new net: F4.2, K2.11
- new net: F3.2, SW1.4
- new net: F5.1, K1.11
- new net 12V: U2.
- new net 12V_ACCESSORIES: K2.14
- new net 12V_CONTROL: K1.A2, K2.A2
- new net 12V_SKIDOO_HARNESS: K1.14
- new net GND: BT1.2 (-), K1.A1, K2.A1
- new net REGULATOR: F2.1
- new net STARTER SOLENOID: F1.1, F2.2, SW1.2
- no-connect marks 0 -> 2

Commit message: Display
Connections:
- net at U1.: now also SW1.3; no longer U2.
- new net: U1., U2.
