File: BMS.kicad_sch (KiCad schematic)
At the start: 3 parts, among them U1 4002

Commit message: Connexion
Parts:
- renumbered D1 to D?, U1 to U?
Changed lines of the file:
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@@
 		(dnp no)
 		(fields_autoplaced yes)
-		(property "Reference" "U?"
+		(property "Reference" "U3"
 			(at 113.665 53.34 0)
 			(effects
@@
 		(dnp no)
 		(fields_autoplaced yes)
-		(property "Reference" "U1"
+		(property "Reference" "U?"
 			(at 111.76 106.68 0)
 			(effects
@@
 		)
 		(instances
+			(project "TEST"
+				(path "/6f31461c-1ce3-4669-a628-d5dc5fed8080/83c1ec6e-e7f8-4b3f-abe9-b7024bdd954a"
+					(reference "U?")
+					(unit 1)
+				)
+			)
 			(project ""
 				(path "/ee56d87b-c754-4edc-93cc-2335df6b1c6f"
@@
 		(dnp no)
 		(fields_autoplaced yes)
-		(property "Reference" "D1"
+		(property "Reference" "D?"
 			(at 164.7825 78.74 0)
 			(effects
@@
 		)
 		(instances
+			(project "TEST"
+				(path "/6f31461c-1ce3-4669-a628-d5dc5fed8080/83c1ec6e-e7f8-4b3f-abe9-b7024bdd954a"
+					(reference "D?")
+					(unit 1)
+				)
+			)
 			(project ""
 				(path "/ee56d87b-c754-4edc-93cc-2335df6b1c6f"

Commit message: BMS5
Parts:
- gave numbers to parts that had none: 2
Connections:
- net GND: now reaches U3.2 (GND)
Changed lines of the file:
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@@
+		)
+	)
+	(hierarchical_label "GND"
+		(shape input)
+		(at 114.3 86.36 270)
+		(effects
+			(font
+				(size 1.27 1.27)
+			)
+			(justify right)
 		)
 	)
@@
 		(dnp no)
 		(fields_autoplaced yes)
-		(property "Reference" "U3"
+		(property "Reference" "U?"
 			(at 113.665 53.34 0)
 			(effects
@@
 		(dnp no)
 		(fields_autoplaced yes)
-		(property "Reference" "U?"
+		(property "Reference" "U1"
 			(at 111.76 106.68 0)
 			(effects
@@
 		(dnp no)
 		(fields_autoplaced yes)
-		(property "Reference" "D?"
+		(property "Reference" "D1"
 			(at 164.7825 78.74 0)
 			(effects

Commit message: Ca marche enfin
Parts:
- renumbered D1 to D?, U1 to U?
Changed lines of the file:
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@@
 		(dnp no)
 		(fields_autoplaced yes)
-		(property "Reference" "U?"
+		(property "Reference" "U3"
 			(at 113.665 53.34 0)
 			(effects
@@
 		(dnp no)
 		(fields_autoplaced yes)
-		(property "Reference" "U1"
+		(property "Reference" "U?"
 			(at 111.76 106.68 0)
 			(effects
@@
 		(dnp no)
 		(fields_autoplaced yes)
-		(property "Reference" "D1"
+		(property "Reference" "D?"
 			(at 164.7825 78.74 0)
 			(effects
