File: DRIVE HV-500.kicad_sch (KiCad schematic)
At the start: 0 parts

Commit message: Drive_Test
Parts:
- added K3: Relay_DPDT, symbol Relay:Relay_DPDT
Connections:
- new net 12V: K3.A2
- new net GND: K3.A1
Changed lines of the file:
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@@
 	(generator_version "9.0")
 	(paper "A4")
+	(wire
+		(pts
+			(xy 99.06 87.63) (xy 106.68 87.63)
+		)
+		(stroke
+			(width 0)
+			(type default)
+		)
+	)
+	(wire
+		(pts
+			(xy 121.92 87.63) (xy 127 87.63)
+		)
+		(stroke
+			(width 0)
+			(type default)
+		)
+	)
+	(hierarchical_label "12V"
+		(shape input)
+		(at 99.06 87.63 180)
+		(effects
+			(font
+				(size 1.27 1.27)
+			)
+			(justify right)
+		)
+	)
+	(hierarchical_label "GND"
+		(shape passive)
+		(at 127 87.63 0)
+		(effects
+			(font
+				(size 1.27 1.27)
+			)
+			(justify left)
+		)
+	)
+	(symbol
+		(lib_id "Relay:Relay_DPDT")
+		(at 114.3 97.79 270)
+		(unit 1)
+		(exclude_from_sim no)
+		(in_bom yes)
+		(on_board yes)
+		(dnp no)
+		(fields_autoplaced yes)
+		(property "Reference" "K3"
+			(at 114.3 77.47 90)
+			(effects
+				(font
+					(size 1.27 1.27)
+				)
+			)
+		)
+		(property "Value" "Relay_DPDT"
+			(at 114.3 80.01 90)
+			(effects
+				(font
+					(size 1.27 1.27)
+				)
+			)
+		)
+		(property "Footprint" ""
+			(at 113.03 114.3 0)
+			(effects
+				(font
+					(size 1.27 1.27)
+				)
+				(justify left)
+				(hide yes)
+			)
+		)
+		(property "Datasheet" "~"
+			(at 114.3 97.79 0)
+			(effects
+				(font
+					(size 1.27 1.27)
+				)
+				(hide yes)
+			)
+		)
+		(property "Description" "Relay DPDT, monostable, EN50005"
+			(at 114.3 97.79 0)
+			(effects
+				(font
+					(size 1.27 1.27)
+				)
+				(hide yes)
+			)
+		)
+		(pin "12"
+		)
+		(pin "A2"
+		)
+		(pin "A1"
+		)
+		(pin "11"
+		)
+		(pin "22"
+		)
+		(pin "21"
+		)
+		(pin "14"
+		)
+		(pin "24"
+		)
+		(instances
+			(project ""
+				(path "/6f31461c-1ce3-4669-a628-d5dc5fed8080/cdf6ae9d-848f-410c-8736-1868ba0a4769"
+					(reference "K3")
+					(unit 1)
+				)
+			)
+		)
+	)
 )
