File: TEST.kicad_sch (KiCad schematic)
At the start: 0 parts

Commit message: Base
Other:
- added sheet BMS (BMS.kicad_sch)
- added sheet DISPLAY (DISPLAY.kicad_sch)
- added sheet DRIVE HV-500 (DRIVE HV-500.kicad_sch)
- added sheet DRIVE HV-550 (DRIVE HV-550.kicad_sch)
- added sheet ECU (ECU.kicad_sch)
- added sheet SKIDOO ELECTRICAL (SKIDOO ELECTRICAL.kicad_sch)
- added sheet Shutdown (Shutdown.kicad_sch)

Commit message: Power Supply
Other:
- sheet SKIDOO ELECTRICAL ports: added 12V, 12V_ACCESSORIES, 12V_CONTROL, GND; removed none
Changed lines of the file:
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@@
 	(sheet
 		(at 80.01 62.23)
-		(size 30.48 21.59)
+		(size 30.48 27.94)
 		(exclude_from_sim no)
 		(in_bom yes)
@@
 		)
 		(property "Sheetfile" "SKIDOO ELECTRICAL.kicad_sch"
-			(at 80.01 84.4046 0)
+			(at 80.01 90.7546 0)
 			(effects
 				(font
@@
 			)
 		)
+		(pin "12V_CONTROL" input
+			(at 80.01 72.39 180)
+			(effects
+				(font
+					(size 1.27 1.27)
+				)
+				(justify left)
+			)
+		)
+		(pin "GND" passive
+			(at 96.4389 90.17 270)
+			(effects
+				(font
+					(size 1.27 1.27)
+				)
+				(justify left)
+			)
+		)
+		(pin "12V" output
+			(at 94.0259 62.23 90)
+			(effects
+				(font
+					(size 1.27 1.27)
+				)
+				(justify right)
+			)
+		)
+		(pin "12V_ACCESSORIES" output
+			(at 99.06 62.23 90)
+			(effects
+				(font
+					(size 1.27 1.27)
+				)
+				(justify right)
+			)
+		)

Commit message: Display
Other:
- sheet DISPLAY ports: added 12V, CAN-B-H, CAN-B-L, GND; removed none
Changed lines of the file:
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@@
+			)
+		)
+		(pin "12V" input
+			(at 88.9 24.13 90)
+			(effects
+				(font
+					(size 1.27 1.27)
+				)
+				(justify right)
+			)
+		)
+		(pin "GND" passive
+			(at 93.98 48.26 270)
+			(effects
+				(font
+					(size 1.27 1.27)
+				)
+				(justify left)
+			)
+		)
+		(pin "CAN-B-L" bidirectional
+			(at 78.74 33.02 180)
+			(effects
+				(font
+					(size 1.27 1.27)
+				)
+				(justify left)
+			)
+		)
+		(pin "CAN-B-H" bidirectional
+			(at 78.74 36.83 180)
+			(effects
+				(font
+					(size 1.27 1.27)
+				)
+				(justify left)
 			)
 		)

Commit message: Connexion
Other:
- sheet BMS ports: added 12V; removed none
Changed lines of the file:
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@@
+			)
+		)
+		(pin "12V" input
+			(at 44.45 62.23 90)
+			(effects
+				(font
+					(size 1.27 1.27)
+				)
+				(justify right)
 			)
 		)

Commit message: Ca marche enfin
Other:
- sheet BMS ports: added GND; removed none
Changed lines of the file:
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@@
 	(generator_version "9.0")
 	(paper "A4")
+	(wire
+		(pts
+			(xy 88.9 16.51) (xy 113.03 16.51)
+		)
+		(stroke
+			(width 0)
+			(type default)
+		)
+	)
+	(wire
+		(pts
+			(xy 88.9 24.13) (xy 88.9 16.51)
+		)
+		(stroke
+			(width 0)
+			(type default)
+		)
+	)
+	(wire
+		(pts
+			(xy 104.14 54.61) (xy 104.14 62.23)
+		)
+		(stroke
+			(width 0)
+			(type default)
+		)
+	)
+	(wire
+		(pts
+			(xy 113.03 54.61) (xy 104.14 54.61)
+		)
+		(stroke
+			(width 0)
+			(type default)
+		)
+	)
+	(wire
+		(pts
+			(xy 113.03 16.51) (xy 113.03 54.61)
+		)
+		(stroke
+			(width 0)
+			(type default)
+		)
+	)
 	(sheet
 		(at 33.02 125.73)
@@
 			)
 		)
+		(pin "GND" input
+			(at 58.42 83.82 270)
+			(effects
+				(font
+					(size 1.27 1.27)
+				)
+				(justify left)
+			)
+		)
 		(instances
 			(project "TEST"
@@
 		)
 		(pin "12V" output
-			(at 94.0259 62.23 90)
-			(effects
-				(font
+			(at 104.14 62.23 90)
+			(effects
+				(font

Commit message: ECU3
Other:
- sheet ECU ports: added 12V, GND; removed none
Changed lines of the file:
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@@
 	(generator_version "9.0")
 	(paper "A4")
+	(junction
+		(at 88.9 16.51)
+		(diameter 0)
+		(color 0 0 0 0)
+	)
+	(wire
+		(pts
+			(xy 45.72 16.51) (xy 88.9 16.51)
+		)
+		(stroke
+			(width 0)
+			(type default)
+		)
+	)
 	(wire
 		(pts
@@
 		(pts
 			(xy 113.03 16.51) (xy 113.03 54.61)
+		)
+		(stroke
+			(width 0)
+			(type default)
+		)
+	)
+	(wire
+		(pts
+			(xy 45.72 24.13) (xy 45.72 16.51)
 		)
 		(stroke
@@
 			)
 		)
+		(pin "12V" input
+			(at 45.72 24.13 90)
+			(effects
+				(font
+					(size 1.27 1.27)
+				)
+				(justify right)
+			)
+		)
+		(pin "GND" passive
+			(at 54.61 48.26 270)
+			(effects
+				(font
+					(size 1.27 1.27)
+				)
+				(justify left)
+			)
+		)

Commit message: Ajout PIN
Other:
- sheet DRIVE HV-500 ports: added 12V, GND; removed none
Changed lines of the file:
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@@
+			)
+		)
+		(pin "12V" input
+			(at 52.07 92.71 90)
+			(effects
+				(font
+					(size 1.27 1.27)
+				)
+				(justify right)
+			)
+		)
+		(pin "GND" passive
+			(at 57.15 116.84 270)
+			(effects
+				(font
+					(size 1.27 1.27)
+				)
+				(justify left)
 			)
 		)
